File: _restore_backup_2026-08-17T17-30-11-840/soundkey.kicad_sch (KiCad schematic)
At the start: 15 parts, among them J1 ISD1820, J2 Conn_01x06_Socket, Q1 AO3401A, U1 XC6206PxxxMR, U2 TP4057, U3 MSM381ACB026

Commit message: 202608171752_new ic
Parts:
- removed C2: 0.1uF, symbol Device:C
- removed C4: 100uF, symbol Device:C_Polarized_US
- removed Q1: AO3401A, Package_TO_SOT_SMD:SOT-23, symbol Transistor_FET:AO3401A
- removed U1: XC6206PxxxMR, Package_TO_SOT_SMD:SOT-23-3, symbol Regulator_Linear:XC6206PxxxMR
- removed U3: MSM381ACB026, symbol 1_New_Library_0:MSM381ACB026
- added Q1: BSS84, Package_TO_SOT_SMD:SOT-23, symbol Transistor_FET:BSS84
Connections:
- net BAT+: now also Q1.3 (D)
- net SP+: no longer J1.9 (SP+)
- net SP-: no longer J1.7 (SP-)
- net VBUS: now also D2.1 (K), Q1.2 (S); no longer C1.1, D1.2 (A), D2.2 (A), J2.2 (Pin_2), R3.2, U2.4 (V_{CC})
- net VCC: now also C1.1, D1.2 (A), D2.2 (A), J2.2 (Pin_2), R3.2, U2.4 (V_{CC}), Q1.1 (G); no longer D2.1 (K)
- no-connect marks 2 -> 1
Other:
- note removed: "isd1820"
- note removed: "mic"
