File: soundkey.kicad_sch (KiCad schematic)
At the start: 15 parts, among them J1 ISD1820, J2 Conn_01x06_Socket, Q1 AO3401A, U1 XC6206PxxxMR, U2 TP4057, U3 MSM381ACB026

Commit message: 2608251535_final-1 sch
Parts:
- removed J1: ISD1820, Package_DIP:DIP-14_W7.62mm_Socket, symbol 1_New_Library_0:ISD1820
- removed MK1: SPH0641LU4H-1, Sensor_Audio:Knowles_LGA-5_3.5x2.65mm, symbol Sensor_Audio:SPH0641LU4H-1
- added C3: 10uF, symbol Device:C
- added C5: 0.1u, symbol Device:C
- added C6, C7: 1uF, symbol Device:C_Small
- added D3: LED, symbol Device:LED
- added J1, J3: Conn_01x01_Socket, symbol Connector:Conn_01x01_Socket
- added R4: 0, symbol Device:R_US
- added R5: 1k, symbol Device:R_US
- added U4: CHR11, Package_SO:SOIC-16_3.9x9.9mm_P1.27mm, symbol 1_New_Library_0:CHR11
Connections:
- net GND is gone; now on net Earth: C1.2, C2.2, C4.2, J2.1 (Pin_1), J2.3 (Pin_3), R1.2, R3.1, U2.2 (GND)
- net SP+: now also U4.14 (SP2)
- net SP-: now also U4.13 (SP1)
- net at U3.1 (VDD): now also C3.1, R4.2
- net M-: now reaches U3.2 (OUT)
- net M-: now also C5.2, U4.7 (M-)
- net Earth: now reaches U3.3 (GND)
- net Earth: now also C3.2, C5.1, C6.1, C7.1, D3.1 (K), U4.12 (GND), U4.8 (SGND)
- new net: C6.2, U4.11 (VMCU)
- new net: D3.2 (A), R5.2
- new net: J1.1 (Pin_1), U4.15 (PLAY), U4.16 (REC)
- new net CH1: U4.4 (CH1)
- new net CH2: R5.1, U4.5 (CH2)
- new net M_VCC: R4.1, U4.6 (M_VCC)
- new net VDDIO: C7.2, J3.1 (Pin_1), U4.10 (VDDIO)
- no-connect marks 2 -> 9
Other:
- note added: "CHR11"
- note added: "LED"
- note added: "SEL"
- note removed: "isd1820"
- moved on the sheet: U1
