File: soundkey.kicad_sch (KiCad schematic)
At the start: 23 parts, among them J1 Conn_01x01_Socket, J2 Conn_01x06_Socket, J3 Conn_01x01_Socket, Q1 AO3401A, U1 XC6206PxxxMR, U2 TP4057, U3 MSM381ACB026, U4 CHR11

Commit message: 2608261612_chg arch.
Parts:
- removed C3: 10uF, symbol Device:C
- removed C5: 0.1u, symbol Device:C
- removed C6, C7: 1uF, symbol Device:C_Small
- removed D3: LED, symbol Device:LED
- removed R5: 1k, symbol Device:R_US
- removed U1: XC6206PxxxMR, Package_TO_SOT_SMD:SOT-23-3, symbol Regulator_Linear:XC6206PxxxMR
- removed U3: MSM381ACB026, symbol 1_New_Library_0:MSM381ACB026
- removed U4: CHR11, Package_SO:SOIC-16_3.9x9.9mm_P1.27mm, symbol 1_New_Library_0:CHR11
- added C3, C4, C5: 0.1uF, symbol Device:C_Small
- added C6: 4.7uF, symbol Device:C_Polarized_Small
- added C8: 22uF, symbol Device:C_Polarized_Small
- added D3: WS2812B, LED_SMD:LED_WS2812B_PLCC4_5.0x5.0mm_P3.2mm, symbol LED:WS2812B
- added J4: ISD1820, Package_DIP:DIP-14_W7.62mm_Socket, symbol 1_New_Library_0:ISD1820
- added MK1: Microphone_Condenser, symbol Device:Microphone_Condenser
- added Q2: AO3401A, Package_TO_SOT_SMD:SOT-23, symbol Transistor_FET:AO3401A
- added R5: 100k, symbol Device:R_Small_US
- added R6: 4.7k, symbol Device:R_US
- added R7: 1k, symbol Device:R_US
- added R8: 100k, symbol Device:R_US
- added R9: 10k, symbol Device:R_Small_US
- added U1: ATtiny85-20P, Package_DIP:DIP-8_W7.62mm, symbol MCU_Microchip_ATtiny:ATtiny85-20P
- J1: value Conn_01x01_Socket -> button-
- J3: value Conn_01x01_Socket -> button+
- R4: value 0 -> 4.7k
- renumbered C4 to C7
Connections:
- net M_VCC is gone; now on net Earth: R4.1
- net Earth: now also J1.1 (Pin_1), C5.2, C6.1, C8.2, D3.3 (VSS), J4.14 (VSS), J4.8 (VSSA), R5.2, U1.4 (GND)
- net SP+: now also J4.9 (SP+)
- net SP-: now also J4.7 (SP-)
- net VCC: now also C5.1, D3.1 (VDD), J4.11 (VCC), Q2.2 (S), R7.2; no longer C2.1, C7.1, D2.1 (K), Q1.2 (S)
- net at R4.2: now also C3.2, MK1.2 (+)
- net VDDIO: no longer names the net of J3.1 (Pin_1)
- net VDDIO: now also U1.2 (XTAL1/PB3)
- new net: R9.1, U1.1 (~{RESET}/PB5)
- new net: C4.2, MK1.1 (-), R6.1
- new net: C8.1, R6.2, R7.1
- new net: J4.10 (ROSC), R5.1
- new net AGC: C6.2, J4.6 (AGC)
- new net DEEPSLP: Q2.1 (G), R8.2, U1.6 (PB1)
- new net LED: D3.4 (DIN), U1.3 (XTAL2/PB4)
- new net MIC: C3.1, J4.4 (MIC)
- new net MICREF: C4.1, J4.5 (MICREF)
- new net PLAYE: J4.2 (PLAYE), U1.5 (AREF/PB0)
- new net REC: J4.1 (REC), U1.7 (PB2)
- new net VSYS: C2.1, C7.1, D2.1 (K), Q1.2 (S), Q2.3 (D), R8.1, R9.2, U1.8 (VCC)
- no-connect marks 9 -> 5
Other:
- note added: "ATtiny"
- note added: "ISD1820"
- note removed: "CHR11"
- note removed: "SEL"
- moved on the sheet: C2, C7, D1, D2, Q1, R1, R2, R3, U2

Commit message: 2608262232_chg arch.
Parts:
- removed J1: button-, symbol Connector:Conn_01x01_Socket
- removed J3: button+, symbol Connector:Conn_01x01_Socket
- added J1: Conn_01x02_Socket, Switch_Keyboard_Kailh:SW_Kailh_KH, symbol Connector:Conn_01x02_Socket
- MK1: footprint (none) -> Sensor_Audio:POM-2244P-C3310-2-R
Connections:
- net Earth: now also J1.2 (Pin_2)
- net at U1.2 (XTAL1/PB3): now also J1.1 (Pin_1)
Other:
- moved on the sheet: C1, J2

Commit message: 2608292346_thisiswild
Parts:
- removed C2: 0.1uF, symbol Device:C
- removed C4: 0.1uF, symbol Device:C_Small
- removed C6: 4.7uF, symbol Device:C_Polarized_Small
- removed C7: 100uF, symbol Device:C_Polarized_US
- removed C8: 22uF, symbol Device:C_Polarized_Small
- removed D1: LED, symbol Device:LED
- removed D3: WS2812B, LED_SMD:LED_WS2812B_PLCC4_5.0x5.0mm_P3.2mm, symbol LED:WS2812B
- removed J4: ISD1820, Package_DIP:DIP-14_W7.62mm_Socket, symbol 1_New_Library_0:ISD1820
- removed MK1: Microphone_Condenser, Sensor_Audio:POM-2244P-C3310-2-R, symbol Device:Microphone_Condenser
- removed R2: 1k, symbol Device:R_US
- removed R4: 4.7k, symbol Device:R_US
- removed R5: 100k, symbol Device:R_Small_US
- removed U1: ATtiny85-20P, Package_DIP:DIP-8_W7.62mm, symbol MCU_Microchip_ATtiny:ATtiny85-20P
- added C10: 10uF, Capacitor_SMD:C_0805_2012Metric, symbol Device:C_Small
- added C11, C14, C2, C7: 100nF, Capacitor_SMD:C_0402_1005Metric, symbol Device:C_Small
- added C12: 10nF, Capacitor_SMD:C_0402_1005Metric, symbol Device:C_Small
- added C13, C9: 1uF, Capacitor_SMD:C_0603_1608Metric, symbol Device:C_Small
- added C15: 470nF, Capacitor_SMD:C_0402_1005Metric, symbol Device:C_Small
- added C16, C4: 10uF, Capacitor_SMD:C_0805_2012Metric, symbol Device:C
- added C6: 22uF, Capacitor_SMD:C_1206_3216Metric, symbol Device:C
- added C8: 10uF, Capacitor_THT:C_Radial_D4.0mm_H5.0mm_P1.50mm, symbol Device:C_Polarized_Small_US
- added D2: WS2812B-2020, LED_SMD:LED_WS2812B-2020_PLCC4_2.0x2.0mm, symbol LED:WS2812B-2020
- added J3: USB_C_Receptacle_USB2.0_16P, Connector_USB:USB_C_Receptacle_GCT_USB4105-xx-A_16P_TopMnt_Horizontal, symbol Connector:USB_C_Receptacle_USB2.0_16P
- added J4: main_Pad, 1_Library:Pad_7_1.5x2.0mm_G2.5mm, symbol Connector:Conn_01x07_Socket
- added J5: UPDI, TestPoint:TestPoint_Pad_D1.0mm, symbol Connector:Conn_01x01_Socket
- added MK1: CMC-4015-40P, 1_Library:MIC_CMC-4015-40P, symbol CMC-4015-40P:CMC-4015-40P
- added R10: 680k, Resistor_SMD:R_0603_1608Metric, symbol Device:R_US
- added R11, R12: 22k, Resistor_SMD:R_0402_1005Metric, symbol Device:R_US
- added R2, R4: 5.1k, Resistor_THT:R_Axial_DIN0204_L3.6mm_D1.6mm_P5.08mm_Horizontal, symbol Device:R_Small_US
- added R5: 2.2k, Resistor_SMD:R_0402_1005Metric, symbol Device:R_US
- added U1: AVR32DU28x-xSTX, Package_DFN_QFN:WQFN-28-1EP_4x4mm_P0.4mm_EP2.7x2.7mm_ThermalVias, symbol 1_New_Library_0:AVR64DU28
- added U3: PAM8301, Package_TO_SOT_SMD:SOT-23-6, symbol Amplifier_Audio:PAM8301
- added U4: TLV9001IDCK, Package_TO_SOT_SMD:SOT-353_SC-70-5, symbol Amplifier_Operational:TLV9001IDCK
- C1: value 1uF -> 100nF; footprint (none) -> Capacitor_SMD:C_0402_1005Metric; now not fitted
- C3, C5: value 0.1uF -> 100nF; footprint (none) -> Capacitor_SMD:C_0402_1005Metric
- D1: renamed from D2; footprint Diode_THT:D_DO-41_SOD81_P10.16mm_Horizontal -> Diode_THT:D_DO-41_SOD81_P7.62mm_Horizontal
- J1: value Conn_01x02_Socket -> button
- J2: value Conn_01x06_Socket -> daughter_Pad; footprint (none) -> 1_Library:Pad_7_1.5x2.0mm_G2.5mm; symbol Connector:Conn_01x06_Socket -> Connector:Conn_01x07_Socket
- R1, R3: footprint (none) -> Resistor_THT:R_Axial_DIN0204_L3.6mm_D1.6mm_P5.08mm_Horizontal
- R6: value 4.7k -> 15k; footprint (none) -> Resistor_SMD:R_0402_1005Metric
- R7: value 1k -> 100k; footprint (none) -> Resistor_SMD:R_0402_1005Metric
- R8: value 100k -> 47k; footprint (none) -> Resistor_SMD:R_0402_1005Metric; now not fitted
- R9: value 10k -> 1k; footprint (none) -> Resistor_SMD:R_0402_1005Metric
Connections:
- net BAT+: now also J2.6 (Pin_6), C16.1; no longer J2.4 (Pin_4)
- net LED: now also D2.3 (DIN), U1.2 (PA4)
- net MIC: now also R10.1, U1.4 (PA6), U4.4; no longer C3.1
- net SP+: now also J4.3 (Pin_3), U3.6 (OUT+); no longer J2.6 (Pin_6)
- net SP-: now also J4.4 (Pin_4), U3.1 (OUT-); no longer J2.5 (Pin_5)
- net VBUS: now also C8.1, J3.A4 (VBUS), J3.A9 (VBUS), J3.B4 (VBUS), J3.B9 (VBUS); no longer C1.1, J2.2 (Pin_2)
- net VCC: now also Q2.3 (D), C10.2, C14.2, C2.2, C6.1, C9.2, D2.4 (VDD), R11.1, R5.1, U3.5 (VDD), U4.5 (V+); no longer C5.1, Q2.2 (S), R7.2
- net VSYS: now also C1.1, C3.2, C5.1, Q2.2 (S), R7.1, C4.1, J4.2 (Pin_2), U1.18 (VDD), U1.24 (VDD); no longer D1.1 (K), Q1.2 (S), Q2.3 (D), R8.1, R9.2
- net at R9.1: now also C11.1, C12.1
- net at J1.1 (Pin_1): now also U1.13 (PD3)
- net at R6.1: now also R10.2, U4.3 (-)
- net at R6.2: now also C7.2; no longer R7.1
- net CHG_sub: now reaches U2.1 (~{CHRG})
- net CHG_sub: now also J2.1 (Pin_1)
- net at U2.6 (PROG): now also R1.2; no longer R1.1
- net DEEPSLP renamed PERIPH_EN_N
- net PERIPH_EN_N: now also R7.2, U1.3 (PA5); no longer R8.2
- removed net Earth: C1.2, C5.2, J1.2 (Pin_2), J2.1 (Pin_1), J2.3 (Pin_3), R1.2, R3.1, U2.2 (GND)
- new net: C13.1, R11.2, R12.1, U4.1 (+)
- new net: C7.1, MK1.P, R5.2
- new net: J3.B5 (CC2), R4.1
- new net: J3.A5 (CC1), R2.2
- new net: J5.1 (Pin_1), U1.23 (PF7/UPDI)
- new net: C15.2, U1.6 (VUSB)
- new net: C11.2, U3.3 (IN)
- new net AUDIN: R9.2, U1.28 (PA2)
- new net CHG: J4.1 (Pin_1), U1.12 (PD2)
- new net D+: J4.7 (Pin_7), U1.8 (DP)
- new net D-: J4.6 (Pin_6), U1.7 (DM)
- new net D_sub+: J2.5 (Pin_5), J3.A6 (D+), J3.B6 (D+)
- new net D_sub-: J2.4 (Pin_4), J3.A7 (D-), J3.B7 (D-)
- new net GND: C1.2, C10.1, C12.2, C13.2, C14.1, C15.1, C2.1, C3.1, C4.2, C5.2, C6.2, C9.1, D2.2 (VSS), J1.2 (Pin_2), J4.5 (Pin_5), MK1.M, R12.2, R8.1, U1.19 (GND), U1.25 (GND), U1.29 (GND_EP), U3.2 (GND), U4.2 (V-)
- new net GND_sub: C16.2, C8.2, J2.2 (Pin_2), J2.7 (Pin_7), J3.A1 (GND), J3.A12 (GND), J3.B1 (GND), J3.B12 (GND), J3.SH (SHIELD), R1.1, R2.1, R3.1, R4.2, U2.2 (GND)
- new net SD_N: R8.2, U1.1 (PA3), U3.4 (~{SD})
- new net VSYS_sub: D1.1 (K), J2.3 (Pin_3), Q1.2 (S)
- no-connect marks 5 -> 19
Other:
- note added: "A close AP to VDD"
- note added: "C0G/NP0 16 V"
- note added: "Low all periph before PA5(HIGH)"
- note added: "PAM8301"
- note added: "X5R 10V"
- note added: "X7R 10V"
- note added: "bat"
- note added: "daughter board"
- note added: "get bat+ from vddbandgap"
- note added: "main"
- note added: "power"
- note added: "res:1% cap no label:X7R 16V"
- note added: "view datasheet 5.2."
- note removed: "ATtiny"
- note removed: "ISD1820"
- note removed: "POWER"
- moved on the sheet: D1, Q1, R3, U2

Commit message: 2608300232_half wire
Parts:
- C11, C7: footprint Capacitor_SMD:C_0402_1005Metric -> Capacitor_SMD:C_0603_1608Metric
- R10: footprint Resistor_SMD:R_0603_1608Metric -> Resistor_SMD:R_0402_1005Metric
Changed lines of the file:
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@@
 			)
 		)
-		(property "Footprint" "Capacitor_SMD:C_0402_1005Metric"
+		(property "Footprint" "Capacitor_SMD:C_0603_1608Metric"
 			(at 40.64 142.24 0)
 			(hide yes)
@@
 			)
 		)
-		(property "Footprint" "Resistor_SMD:R_0603_1608Metric"
+		(property "Footprint" "Resistor_SMD:R_0402_1005Metric"
 			(at 83.566 151.384 90)
 			(hide yes)
@@
 			)
 		)
-		(property "Footprint" "Capacitor_SMD:C_0402_1005Metric"
+		(property "Footprint" "Capacitor_SMD:C_0603_1608Metric"
 			(at 205.74 135.89 0)
 			(hide yes)

Commit message: 2608301213_drcing
Connections:
- net at U1.13 (PD3): no longer J1.1 (Pin_1)
- net at U1.14 (PD4): now also J1.1 (Pin_1)
Other:
- moved on the sheet: J1
Changed lines of the file:
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@@
 	)
 	(no_connect
+		(at 203.2 64.77)
+	)
+	(no_connect
 		(at 203.2 48.26)
 	)
@@
 	)
 	(no_connect
-		(at 203.2 67.31)
-	)
-	(no_connect
 		(at 203.2 69.85)
 	)
@@
 	(wire
 		(pts
+			(xy 191.77 67.31) (xy 203.2 67.31)
+		)
+		(stroke
+			(width 0)
+			(type default)
+		)
+	)
+	(wire
+		(pts
 			(xy 118.11 49.53) (xy 138.43 49.53)
 		)
@@
 	(wire
 		(pts
-			(xy 194.31 64.77) (xy 203.2 64.77)
-		)
-		(stroke
-			(width 0)
-			(type default)
-		)
-	)
-	(wire
-		(pts
 			(xy 85.09 106.68) (xy 85.09 107.95)
 		)
@@
 	(symbol
 		(lib_id "Connector:Conn_01x02_Socket")
-		(at 189.23 64.77 0)
+		(at 186.69 67.31 0)
 		(mirror y)
 		(unit 1)
@@
 		(dnp no)
 		(property "Reference" "J1"
-			(at 189.865 72.39 0)
+			(at 187.325 74.93 0)
 			(show_name no)
 			(do_not_autoplace no)
@@
 		)
 		(property "Value" "button"
-			(at 189.865 69.85 0)
+			(at 187.325 72.39 0)
 			(show_name no)
 			(do_not_autoplace no)
@@
 		)
 		(property "Footprint" "Switch_Keyboard_Kailh:SW_Kailh_KH"
-			(at 189.23 64.77 0)
+			(at 186.69 67.31 0)
 			(hide yes)
 			(show_name no)
@@
 		)
 		(property "Datasheet" ""
-			(at 189.23 64.77 0)
+			(at 186.69 67.31 0)
 			(hide yes)
 			(show_name no)
@@
 		)
 		(property "Description" "Generic connector, single row, 01x02, script generated"
-			(at 189.23 64.77 0)
+			(at 186.69 67.31 0)
 			(hide yes)
 			(show_name no)
@@
 		)
 		(property "Sim.Pins" ""
-			(at 189.23 64.77 0)
+			(at 186.69 67.31 0)
 			(hide yes)
 			(show_name no)
@@
 	(symbol
 		(lib_id "power:GND")
-		(at 194.31 67.31 90)
+		(at 191.77 69.85 90)
 		(unit 1)
 		(body_style 1)
@@
 		(fields_autoplaced yes)
 		(property "Reference" "#PWR11"
-			(at 200.66 67.31 0)
+			(at 198.12 69.85 0)
 			(hide yes)
 			(show_name no)
@@
 		)
 		(property "Value" "GND"
-			(at 198.12 67.3099 90)
+			(at 195.58 69.8499 90)
 			(show_name no)
 			(do_not_autoplace no)
@@
 		)
 		(property "Footprint" ""
-			(at 194.31 67.31 0)
+			(at 191.77 69.85 0)
 			(hide yes)
 			(show_name no)
@@
 		)
 		(property "Datasheet" ""
-			(at 194.31 67.31 0)
+			(at 191.77 69.85 0)
 			(hide yes)
 			(show_name no)
@@
 		)
 		(property "Description" "Power symbol creates a global label with name \"GND\" , ground"
-			(at 194.31 67.31 0)
+			(at 191.77 69.85 0)
 			(hide yes)
 			(show_name no)

Commit message: 2608310153_ready for vcut
Parts:
- U1: footprint Package_DFN_QFN:WQFN-28-1EP_4x4mm_P0.4mm_EP2.7x2.7mm_ThermalVias -> 1_Library:VQFN-28-1EP_4x4mm_P0.4mm_EP2.7x2.7mm_ThermalVias
Changed lines of the file:
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@@
 	(wire
 		(pts
+			(xy 226.06 83.82) (xy 226.06 87.63)
+		)
+		(stroke
+			(width 0)
+			(type default)
+		)
+	)
+	(wire
+		(pts
 			(xy 72.39 142.24) (xy 73.66 142.24)
 		)
@@
 	(wire
 		(pts
+			(xy 226.06 87.63) (xy 223.52 87.63)
+		)
+		(stroke
+			(width 0)
+			(type default)
+		)
+	)
+	(wire
+		(pts
 			(xy 222.25 129.54) (xy 222.25 123.19)
 		)
@@
 		(in_pos_files yes)
 		(dnp no)
-		(fields_autoplaced yes)
 		(property "Reference" "U1"
-			(at 225.6633 83.82 0)
+			(at 226.822 84.074 0)
 			(show_name no)
 			(do_not_autoplace no)
@@
 		)
 		(property "Value" "AVR32DU28x-xSTX"
-			(at 225.6633 86.36 0)
+			(at 226.822 86.36 0)
 			(show_name no)
 			(do_not_autoplace no)
@@
 			)
 		)
-		(property "Footprint" "Package_DFN_QFN:WQFN-28-1EP_4x4mm_P0.4mm_EP2.7x2.7mm_ThermalVias"
+		(property "Footprint" "1_Library:VQFN-28-1EP_4x4mm_P0.4mm_EP2.7x2.7mm_ThermalVias"
 			(at 223.52 58.42 0)
 			(hide yes)
