File: soundkey.kicad_pcb (KiCad board)
At the start: 2 copper layers, 5 parts, among them J1 ISD1820, Q1 BSS84, U2 TP4057

Commit message: 2608262232_chg arch.
Parts:
- added D3: WS2812B, LED_SMD:LED_WS2812B_PLCC4_5.0x5.0mm_P3.2mm, F.Cu at (181.5, 112.7)
- added J4: ISD1820, Package_DIP:DIP-14_W7.62mm_Socket, F.Cu at (153.2, 97.0)
- added Q2: AO3401A, Package_TO_SOT_SMD:SOT-23, F.Cu at (169.9, 118.4)
- added U1: ATtiny85-20P, Package_DIP:DIP-8_W7.62mm, F.Cu at (164.5, 96.9)
- J1: value ISD1820 -> Conn_01x02_Socket; footprint Package_DIP:DIP-14_W7.62mm_Socket -> Switch_Keyboard_Kailh:SW_Kailh_KH
- MK1: value SPH0641LU4H-1 -> Microphone_Condenser; footprint Sensor_Audio:Knowles_LGA-5_3.5x2.65mm -> Sensor_Audio:POM-2244P-C3310-2-R
- Q1: value BSS84 -> AO3401A
- moved MK1 66.0 mm to (187.2, 104.2)
- moved J1 53.6 mm to (183.0, 91.3)
- moved Q1 29.9 mm to (150.3, 120.8)
- moved D2 28.6 mm to (157.3, 89.0)
- moved U2 6.85 mm to (148.6, 88.8)
Connections:
- D2 pad 1: /VBUS -> /VSYS
- D2 pad 2: /VCC -> /VBUS
- J1 pad 1: unconnected-(J1-REC-Pad1) -> Net-(J1-Pin_1)
- J1 pad 2: unconnected-(J1-PLAYE-Pad2) -> Earth
- MK1 pad 1: unconnected-(MK1-DATA-Pad1) -> Net-(MK1--)
- MK1 pad 2: unconnected-(MK1-SEL-Pad2) -> Net-(MK1-+)
- Q1 pad 1: /VCC -> /VBUS
- Q1 pad 2: /VBUS -> /VSYS
- U2 pad 2: GND -> Earth
- U2 pad 4: /VCC -> /VBUS

Commit message: 2608292346_thisiswild
Parts:
- removed D3: WS2812B, LED_SMD:LED_WS2812B_PLCC4_5.0x5.0mm_P3.2mm
- added C10: 10uF, Capacitor_SMD:C_0805_2012Metric, F.Cu at (139.3, 154.2)
- added C11: 100nF, Capacitor_SMD:C_0402_1005Metric, F.Cu at (138.3, 157.9)
- added C12: 10nF, Capacitor_SMD:C_0402_1005Metric, F.Cu at (138.3, 156.1)
- added C13: 1uF, Capacitor_SMD:C_0603_1608Metric, F.Cu at (140.1, 160.0)
- added C14: 100nF, Capacitor_SMD:C_0402_1005Metric, B.Cu at (144.0, 162.7)
- added C15: 470nF, Capacitor_SMD:C_0402_1005Metric, F.Cu at (143.7, 164.8)
- added C2: 100nF, Capacitor_SMD:C_0402_1005Metric, F.Cu at (142.0, 160.2)
- added C3: 100nF, Capacitor_SMD:C_0402_1005Metric, F.Cu at (146.9, 160.2)
- added C4: 10uF, Capacitor_SMD:C_0805_2012Metric, F.Cu at (134.7, 148.8)
- added C5: 100nF, Capacitor_SMD:C_0402_1005Metric, F.Cu at (150.1, 163.2)
- added C7: 100nF, Capacitor_SMD:C_0402_1005Metric, F.Cu at (137.7, 163.1)
- added C8: 10uF, Capacitor_THT:C_Radial_D4.0mm_H5.0mm_P1.50mm, F.Cu at (120.8, 156.7)
- added C9: 1uF, Capacitor_SMD:C_0603_1608Metric, F.Cu at (136.1, 154.5)
- added D2: WS2812B-2020, LED_SMD:LED_WS2812B-2020_PLCC4_2.0x2.0mm, B.Cu at (144.1, 160.7)
- added J2: daughter_Pad, 1_Library:Pad_7_1.5x2.0mm_G2.5mm, F.Cu at (114.6, 148.7)
- added J3: USB_C_Receptacle_USB2.0_16P, Connector_USB:USB_C_Receptacle_GCT_USB4105-xx-A_16P_TopMnt_Horizontal, F.Cu at (114.6, 165.2)
- added J5: UPDI, TestPoint:TestPoint_Pad_D1.0mm, F.Cu at (150.1, 157.8)
- added R1: 15k, Resistor_THT:R_Axial_DIN0204_L3.6mm_D1.6mm_P5.08mm_Horizontal, F.Cu at (117.6, 157.0)
- added R10: 680k, Resistor_SMD:R_0603_1608Metric, F.Cu at (141.3, 164.1)
- added R11: 22k, Resistor_SMD:R_0402_1005Metric, F.Cu at (137.7, 161.2)
- added R12: 22k, Resistor_SMD:R_0402_1005Metric, F.Cu at (137.7, 160.2)
- added R2: 5.1k, Resistor_THT:R_Axial_DIN0204_L3.6mm_D1.6mm_P5.08mm_Horizontal, F.Cu at (107.2, 159.1)
- added R3: 100k, Resistor_THT:R_Axial_DIN0204_L3.6mm_D1.6mm_P5.08mm_Horizontal, F.Cu at (112.5, 154.9)
- added R4: 5.1k, Resistor_THT:R_Axial_DIN0204_L3.6mm_D1.6mm_P5.08mm_Horizontal, F.Cu at (117.0, 159.3)
- added R5: 2.2k, Resistor_SMD:R_0402_1005Metric, F.Cu at (137.7, 162.1)
- added R6: 15k, Resistor_SMD:R_0402_1005Metric, F.Cu at (138.9, 164.0)
- added R7: 100k, Resistor_SMD:R_0402_1005Metric, F.Cu at (137.4, 149.4)
- added R9: 1k, Resistor_SMD:R_0402_1005Metric, F.Cu at (139.2, 157.0)
- added U3: PAM8301, Package_TO_SOT_SMD:SOT-23-6, F.Cu at (136.1, 157.3)
- added U4: TLV9001IDCK, Package_TO_SOT_SMD:SOT-353_SC-70-5, F.Cu at (141.4, 162.2)
- D1: renamed from D2; footprint Diode_THT:D_DO-41_SOD81_P10.16mm_Horizontal -> Diode_THT:D_DO-41_SOD81_P7.62mm_Horizontal
- J1: value Conn_01x02_Socket -> button; moved to B.Cu
- J4: value ISD1820 -> main_Pad; footprint Package_DIP:DIP-14_W7.62mm_Socket -> 1_Library:Pad_7_1.5x2.0mm_G2.5mm
- MK1: value Microphone_Condenser -> CMC-4015-40P; footprint Sensor_Audio:POM-2244P-C3310-2-R -> 1_Library:MIC_CMC-4015-40P; moved to B.Cu
- U1: value ATtiny85-20P -> AVR32DU28x-xSTX; footprint Package_DIP:DIP-8_W7.62mm -> Package_DFN_QFN:WQFN-28-1EP_4x4mm_P0.4mm_EP2.7x2.7mm_ThermalVias
- moved U2 78.0 mm to (109.4, 156.3)
- moved J1 77.5 mm to (142.0, 157.0), turned to 180 degrees
- moved D1 77.3 mm to (111.8, 151.5)
- moved MK1 74.8 mm to (139.8, 162.1), turned to 180 degrees
- moved U1 68.7 mm to (146.9, 163.3)
- moved J4 64.4 mm to (133.3, 158.2), turned to -90 degrees
- moved Q1 52.8 mm to (108.4, 152.8), turned to 180 degrees
- moved Q2 47.5 mm to (136.1, 151.8), turned to -90 degrees
Connections:
- D1 pad 1: /VSYS -> /VSYS_sub
- J1 pad 2: Earth -> GND
- J4 pad 1: /REC -> /CHG
- J4 pad 2: /PLAYE -> VSYS
- J4 pad 3: unconnected-(J4-PLAYL-Pad3) -> /SP+
- J4 pad 4: /MIC -> /SP-
- J4 pad 5: /MICREF -> GND
- J4 pad 6: /AGC -> /D-
- J4 pad 7: /SP- -> /D+
- Q1 pad 2: /VSYS -> /VSYS_sub
- Q2 pad 1: /DEEPSLP -> /PERIPH_EN_N
- Q2 pad 2: /VCC -> VSYS
- Q2 pad 3: /VSYS -> VCC
- U1 pad 1: Net-(U1-~{RESET}/PB5) -> /SD_N
- U1 pad 2: Net-(J1-Pin_1) -> /LED
- U1 pad 3: /LED -> /PERIPH_EN_N
- U1 pad 4: Earth -> /MIC
- U1 pad 5: /PLAYE -> unconnected-(U1-PA7-Pad5)
- U1 pad 6: /DEEPSLP -> Net-(U1-VUSB)
- U1 pad 7: /REC -> /D-
- U1 pad 8: /VSYS -> /D+
- U2 pad 1: Net-(U2-~{CHRG}) -> /CHG_sub
- U2 pad 2: Earth -> GND_sub
Routing:
- net /VBUS: track 0.00 -> 46.2 mm, vias 0 -> 2
- net /BAT+: track 0.00 -> 24.8 mm, vias 0 -> 2
- net /D_sub+: track 0.00 -> 15.9 mm
- net /D_sub-: track 0.00 -> 15.9 mm
- net /CHG_sub: track 0.00 -> 7.35 mm
- net GND: track 0.00 -> 6.77 mm
- net Net-(U4-+): track 0.00 -> 6.28 mm
- net /VSYS_sub: track 0.00 -> 5.47 mm
- net Net-(J3-CC1): track 0.00 -> 2.94 mm
- net Net-(U2-PROG): track 0.00 -> 2.94 mm
- net Net-(C7-Pad1): track 0.00 -> 2.71 mm
- net VSYS: track 0.00 -> 2.52 mm
- net Net-(J3-CC2): track 0.00 -> 2.51 mm
- net Net-(U4--): track 0.00 -> 2.33 mm
- net VCC: track 0.00 -> 1.93 mm
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- added copper zone on B.Cu, net GND
- added copper zone on F.Cu, net GND
- added copper zone on B.Cu, net GND_sub
- added copper zone on F.Cu, net GND_sub
Other:
- board outline added: 45.9 x 20.5 mm

Commit message: 2608300232_half wire
Parts:
- C11, C7: footprint Capacitor_SMD:C_0402_1005Metric -> Capacitor_SMD:C_0603_1608Metric
- R10: footprint Resistor_SMD:R_0603_1608Metric -> Resistor_SMD:R_0402_1005Metric
- moved C11 1.41 mm to (139.0, 159.1), turned to 180 degrees
- moved R6 1.32 mm to (140.1, 164.5)
- moved C2 0.88 mm to (142.7, 160.8)
- moved MK1 0.88 mm to (140.4, 162.6)
- moved C13 0.88 mm to (140.8, 160.5)
- moved U4 0.88 mm to (142.1, 162.8)
- moved R10 0.75 mm to (142.0, 164.4)
- moved R11 0.71 mm to (138.3, 161.4)
- moved R12 0.71 mm to (138.3, 160.4)
- moved R5 0.69 mm to (138.3, 162.3)
- moved C7 0.48 mm to (137.7, 163.5)
- moved C15 0.37 mm to (143.3, 164.6)
- moved R9 0.17 mm to (139.2, 157.2)
Routing:
- net VSYS: track 2.52 -> 15.9 mm
- net VCC: track 1.93 -> 7.53 mm
- net /SP-: track 0.00 -> 2.18 mm
- net /SP+: track 0.16 -> 2.02 mm
- net Net-(U1-VUSB): track 0.00 -> 1.62 mm
- net Net-(C7-Pad2): track 1.56 -> 3.08 mm
- net Net-(U3-IN): track 0.00 -> 1.49 mm
- net Net-(C7-Pad1): track 2.71 -> 3.52 mm

Commit message: 2608301213_drcing
Parts:
- moved J5 2.27 mm to (149.0, 159.8)
- moved D2 1.89 mm to (144.3, 162.6)
- moved C14 1.87 mm to (143.9, 164.6)
- moved R2 0.47 mm to (107.6, 159.1)
- moved R4 0.43 mm to (116.6, 159.3)
- moved D1 0.21 mm to (111.7, 151.6)
- moved J2 0.19 mm to (114.6, 148.9)
Connections:
- U1 pad 13: Net-(J1-Pin_1) -> unconnected-(U1-PD3-Pad13)
- U1 pad 14: unconnected-(U1-PD4-Pad14) -> Net-(J1-Pin_1)
Routing:
- net /CHG: track 0.00 -> 33.3 mm, vias 0 -> 2
- net VCC: track 7.53 -> 32.1 mm, vias 0 -> 3
- net /PERIPH_EN_N: track 0.00 -> 19.4 mm
- net /SD_N: track 0.00 -> 16.9 mm, vias 0 -> 1
- net Net-(J1-Pin_1): track 0.00 -> 13.8 mm, vias 0 -> 1
- net /D+: track 0.00 -> 13.6 mm
- net /D-: track 0.00 -> 13.5 mm
- net /AUDIN: track 0.00 -> 12.8 mm, vias 0 -> 2
- net /BAT+: track 24.8 -> 28.1 mm
- net Net-(C11-Pad1): track 0.00 -> 3.15 mm
- net VSYS: track 15.9 -> 18.4 mm
- net Net-(J5-Pin_1): track 0.00 -> 2.21 mm
- net /MIC: track 1.12 -> 3.21 mm
- net GND: track 6.77 -> 8.42 mm, vias 0 -> 6

Commit message: 2608310153_ready for vcut
Parts:
- U1: footprint Package_DFN_QFN:WQFN-28-1EP_4x4mm_P0.4mm_EP2.7x2.7mm_ThermalVias -> 1_Library:VQFN-28-1EP_4x4mm_P0.4mm_EP2.7x2.7mm_ThermalVias
- moved R4 7.57 mm to (124.2, 158.8)
- moved U2 7.57 mm to (117.0, 155.9)
- moved R1 7.57 mm to (125.1, 156.5)
- moved R2 7.57 mm to (115.2, 158.7)
- moved R3 7.57 mm to (120.0, 154.4)
- moved C8 7.57 mm to (128.3, 156.2)
- moved J2 7.57 mm to (122.2, 148.5)
- moved D1 7.57 mm to (119.2, 151.2)
- moved J3 7.57 mm to (122.2, 164.8)
- moved Q1 7.54 mm to (115.9, 152.3)
- moved C11 3.44 mm to (135.9, 160.5)
- moved C12 1.87 mm to (138.3, 158.0)
- moved R9 1.71 mm to (139.3, 158.9), turned to -90 degrees
- moved C15 0.56 mm to (143.8, 164.3), turned to 0 degrees
- moved C3 0.44 mm to (147.3, 160.2)
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Routing:
- net VSYS: track 18.4 -> 38.3 mm
- net /LED: track 0.00 -> 7.94 mm, vias 0 -> 1
- net /AUDIN: track 12.8 -> 8.54 mm, vias 2 -> 0
- net /BAT+: track 28.1 -> 25.4 mm
- net /PERIPH_EN_N: track 19.4 -> 21.5 mm, vias 0 -> 2
- net Net-(U3-IN): track 1.49 -> 3.07 mm
- net Net-(U4-+): track 5.95 -> 4.59 mm
- net GND: track 8.42 -> 9.55 mm, vias 6 -> 23
- net Net-(J1-Pin_1): track 13.8 -> 14.6 mm
- net /CHG: track 33.3 -> 34.1 mm
- net Net-(C11-Pad1): track 3.15 -> 3.92 mm
- net /D-: track 13.5 -> 14.3 mm
- net /D+: track 13.6 -> 14.3 mm
- net VCC: track 32.1 -> 32.8 mm
- net /MIC: track 3.21 -> 3.71 mm
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Other:
- board size 45.9 x 20.5 mm -> 38.3 x 20.1 mm

Commit message: 2608310324_ready for produce(vcut canceled)
Parts:
- moved R6 5.65 mm to (145.7, 164.7)
- moved C14 5.64 mm to (149.4, 164.8)
- moved C5 5.64 mm to (156.2, 163.3)
- moved D2 5.64 mm to (149.7, 162.7)
- moved J4 5.64 mm to (138.9, 158.4)
- moved C10 5.64 mm to (144.9, 154.3)
- moved C11 5.64 mm to (141.5, 160.6)
- moved C12 5.64 mm to (144.0, 158.1)
- moved C13 5.64 mm to (146.4, 160.7)
- moved C15 5.64 mm to (149.5, 164.5)
- moved C2 5.64 mm to (148.3, 160.9)
- moved C3 5.64 mm to (153.0, 160.4)
- moved C4 5.64 mm to (140.4, 148.9)
- moved C7 5.64 mm to (143.3, 164.0)
- moved C9 5.64 mm to (141.7, 154.7)
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Other:
- board size 38.3 x 20.1 mm -> 46.7 x 20.3 mm
